File: projects/helm-controller/pcb/helm-controller.kicad_sch (KiCad schematic)
At the start: 408 parts, among them J1 Optional Bond, J2 Future Use, J3 Conn_01x02_Pin, Q1 DMN6075S, Q10 DMN6075S, Q11 BSS314PE, Q12 DMN6075S, Q13 BSS314PE, Q14 DMN6075S, Q15 DMN6075S, Q2 BSS314PE, Q3 DMN6075S, Q4 BSS314PE, Q5 DMN6075S, Q6 DMN6075S, Q7 DMN6075S, Q8 DMN6075S, Q9 BSS314PE, SW1 Boot, SW2 Reset, T1 760390014, T2 760390014

Commit message: Bumped the version to 1.8.0 and updated the project name.
Swapped 0.1uF THT caps for SMD

Signed-off-by: digimer <digital.mermaid@gmail.com>
Other:
- company: The Digital Mermaid -> Tuskar Marine
- title: Main Control Unit -> Helm Controller

Commit message: Just starting the conversion from THT / D-Sub, much worth still to be done.
Signed-off-by: digimer <digital.mermaid@gmail.com>
Parts:
- removed DA1: L17H2330131, mr-stuff:Amphenol_L17H2330131, symbol mr-parts:DA15_Pins_Stacked
- removed DA2: L17H2440131, mr-stuff:Amphenol_L17H2440131, symbol mr-parts:DA15_Sockets_Stacked
- removed DB1: L17H2660131, mr-stuff:Amphenol_L17H2660131, symbol mr-parts:DB25_Sockets_Stacked
- removed DE2: L777SDE09PA4CH4F, mr-stuff:Amphenol L777SDE09PA4CH4F, symbol mr-parts:Amphenol L777SDE09PA4CH4F
- C1, C12, C13, C14, C15, C16, C17, C19, C2, C20, C25, C26, C27, C28, C29, C30, C31, C32, C33, C34, C35, C36, C37, C38, C41, C45, C47, C48, C49, C5, C50, C51, C52, C53, C54, C55, C56, C57, C58, C59, C60, C61, C62, C63, C64, C65, C66, C67, C68, C69, C70, C71, C72, C73, C74, C75, C76, C77, C78, C79, C80, C81, C82, C89, C90: symbol Device:C -> mr-parts:Kyocera 08051C104K4Z2A
