File: projects/n2k-transceiver/N2K Transceiver.kicad_pcb (KiCad board)
At the start: 4 copper layers, 60 x 75 mm, 77 parts, among them J1 JTAG, SW1 SW_MEC_5G, SW2 SW_MEC_5G, SW3 SW_MEC_5G

Commit message: Standadized LEDs and GPIO resistors.
* Settled on 475 Ohm current limiting resistors for GPIO.
* Settled on Vishay TLMS1101-GS15 SMD LEDs.
* Added an LED to the Masthead controller for various status applications.

Signed-off-by: digimer <digital.mermaid@gmail.com>
Parts:
- added C64: 0.1uF, mr-stuff:Kyocera AVX 0805, F.Cu at (157.9, 65.4)
- added C65: 0.1uF, mr-stuff:Kyocera AVX 0805, F.Cu at (157.9, 68.5)
- added R52: 475R, mr-stuff:Stackpole RNCP0805, F.Cu at (113.5, 58.4)
- added R53: 475R, mr-stuff:Stackpole RNCP0805, F.Cu at (153.4, 60.7)
- added R54: 10kR, mr-stuff:Stackpole RNCP0805, F.Cu at (153.4, 63.6)
- added SW4: SW_MEC_5G, mr-stuff:SW_TS03-66-50-BK-160-LCR-D-67, F.Cu at (111.5, 73.1)
- R21, R22, R23, R25, R26, R27, R28: value 681R -> 475R; footprint mr-stuff:Stackpole RMCA0805 -> mr-stuff:Stackpole RNCP0805
- moved R24 39.4 mm to (151.8, 66.9)
Connections:
- MCU1 pad 20: unconnected-(MCU1-IO12-Pad20) -> /CONFIG_SW
- R24 pad 1: /LED_ENABLE -> Net-(R24-Pad1)
- SW3 pad 1: /LED_ENABLE -> Net-(R24-Pad1)
- SW3 pad 2: /LED_ENABLE -> Net-(R24-Pad1)
- SW3 pad 3: GND -> Net-(C64-Pad1)
- SW3 pad 4: GND -> Net-(C64-Pad1)
Routing:
- net /LED_ENABLE: track 39.0 -> 22.2 mm
- net Net-(R24-Pad1): track 0.00 -> 7.68 mm, vias 0 -> 1
- net +3.3V: track 74.0 -> 72.6 mm, vias 14 -> 13
Other:
- board text added: "N2K Transceiver v1.0.0 - 2026 MRGN-xxxx Rev. A"
- board text added: "© Tuskar Marine - CERN-OHL-W-2.0"
- board text removed: "-=] License CERN OHL-WR Ver. 2"
- board text removed: "N2K Transceiver © Tuskar Marine v1.0.0 - 2026 Prototype"
