File: projects/masthead-controller/pcb/Masthead Controller.kicad_pcb (KiCad board)
At the start: 4 copper layers, 150 x 83 mm, 228 parts, among them Q1 2N7002, Q2 2N7002, Q3 BSS138P,215, Q4 BSS138P,215, SW1 SW_MEC_5G, SW2 SW_MEC_5G, SW3 SW_MEC_5G

Commit message: Changed spreader lights to fail-off.
Signed-off-by: digimer <digital.mermaid@gmail.com>
Parts:
- added R74: 4.7kR, mr-stuff:Stackpole RMCA0805, F.Cu at (182.9, 107.6)
- added R76: 4.7kR, mr-stuff:Stackpole RMCA0805, F.Cu at (189.8, 107.6)
Routing:
- net GND: track 262.7 -> 275.7 mm
- net /DECK_PRI_JPR: track 68.1 -> 71.3 mm, vias 0 -> 2
- net /DECK_SEC_JPR: track 79.9 -> 82.4 mm
