File: projects/usb-c-pd-x2/USB-C PD x2.kicad_pcb (KiCad board)
At the start: 4 copper layers, 96 x 136 mm, 161 parts, among them J1 Conn_02x05_Odd_Even, J2 Conn_01x05_Pin

Commit message: Removed the polygon pours from the TVS1.
Prototype showed the heat leeching was too much to reasonable solder. The 2mm traces should be sufficient ampacity for a transient event.

Signed-off-by: digimer <digital.mermaid@gmail.com>
Routing:
- net Net-(HS1-D): track 47.8 -> 56.7 mm, vias 28 -> 22
- net -BATT: track 99.3 -> 105.5 mm
