File: projects/usb-c-pd-x2/pcb/USB-C PD x2.kicad_pcb (KiCad board)
At the start: 4 copper layers, 96 x 136 mm, 161 parts, among them J1 Conn_02x05_Odd_Even, J2 Conn_01x05_Pin

Commit message: Updated F.Silkscreen ID data, set v1.3.3
Signed-off-by: digimer <digital.mermaid@gmail.com>
Other:
- board text added: "USB-C PD 2x 100w v1.3.3 - 2026 MRGN-0011 Rev. A"
- board text added: "© Tuskar Marine - CERN-OHL-W-2.0"
- board text removed: "-=] License CERN Open Hardware Licence Weakly Reciprocal Version 2"
- board text removed: "USB-C PD Dual Channel 100w v1.3.3 - Prototype - 01 © The Digital Mermaid - 2026"
Changed lines of the file:
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@@
 	(title_block
 		(title "USB-C PD 2x 100W")
-		(date "2026-08-13")
+		(date "2026-09-30")
 		(rev "v1.3.3")
-		(company "The Digital Mermaid")
+		(company "Tuskar Marine")
 	)
 	(layers
@@
 		(layer "Edge.Cuts")
 	)
-	(gr_text "USB-C PD Dual Channel 100w\nv1.3.3 - Prototype - 01\n© The Digital Mermaid - 2026"
-		(at 88.4 63.4 0)
+	(gr_text "USB-C PD 2x 100w\nv1.3.3 - 2026\nMRGN-0011 Rev. A"
+		(at 100 52 0)
 		(layer "F.SilkS")
 		(effects
@@
 				(thickness 0.15)
 			)
-			(justify left)
+			(justify top)
 		)
 	)
-	(gr_text "-=] License\nCERN Open Hardware Licence\nWeakly Reciprocal\nVersion 2"
-		(at 88.6 56 0)
+	(gr_text "© Tuskar Marine - CERN-OHL-W-2.0\n"
+		(at 100 58 0)
 		(layer "F.SilkS")
 		(effects
@@
 				(thickness 0.15)
 			)
-			(justify left)
+			(justify top)
 		)
 	)
@@
 		)
 	)
+	(barcode
+		(at 100 66 0)
+		(layer "F.SilkS")
+		(size 10 10)
+		(text "HTTPS://TSUKAR.CA/S/MRGN-0011-A")
+		(text_height 1.5)
+		(type qr)
+		(ecc_level M)
+		(hide yes)
+		(knockout no)
+	)
 	(segment
