File: projects/usb-c-pd-x2/pcb/USB-C PD x2.kicad_sch (KiCad schematic)
At the start: 160 parts, among them J1 Conn_02x05_Odd_Even, J2 Conn_01x05_Pin

Commit message: Started converting Helm Controller to SMD
Signed-off-by: digimer <digital.mermaid@gmail.com>
Parts:
- PD1: symbol mr-parts:Infineon_CYPD7272 -> mr-parts:Infineon CYPD727268LQXQXQSA1
Changed lines of the file:
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@@
 	)
 	(symbol
-		(lib_id "mr-parts:Infineon_CYPD7272")
+		(lib_id "mr-parts:Infineon CYPD727268LQXQXQSA1")
 		(at 339.09 101.6 0)
 		(unit 1)
@@
 			(hide yes)
 			(show_name no)
-			(do_not_autoplace no)
-			(effects
-				(font
-					(size 1.27 1.27)
-				)
-			)
-		)
-		(property "Sim.Pins" ""
-			(at 339.09 101.6 0)
-			(hide yes)
-			(show_name no)
