File: projects/helm-controller/Main Control Unit.kicad_pcb (KiCad board)
At the start: 4 copper layers, 280 x 200 mm, 409 parts, among them J1 Optional Bond, J2 Future Use, J3 Conn_01x02_Pin, Q1 DMN6075S, Q10 DMN6075S, Q11 BSS314PE, Q12 DMN6075S, Q13 BSS314PE, Q14 DMN6075S, Q15 DMN6075S, Q2 BSS314PE, Q3 DMN6075S, Q4 BSS314PE, Q5 DMN6075S, Q6 DMN6075S, Q7 DMN6075S, Q8 DMN6075S, Q9 BSS314PE, SW1 Boot, SW2 Reset, T1 760390014, T2 760390014

Commit message: Started converting Helm Controller to SMD
Signed-off-by: digimer <digital.mermaid@gmail.com>
Changed lines of the file:
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@@
 			)
 		)
-		(property "Datasheet" "https://assets.nexperia.com/documents/data-sheet/PZUXB_SER.pdf"
+		(property "Datasheet" ""
 			(at 0 0 90)
 			(unlocked yes)
@@
 			)
 		)
-		(property "Description" "Zener Diode 15 V 310 mW ±2% Surface Mount SOD-323F"
+		(property "Description" ""
 			(at 0 0 90)
 			(unlocked yes)
@@
 			)
 		)
-		(property "Part" "Nexperia PZU15B2,115"
-			(at 0 0 90)
-			(unlocked yes)
-			(layer "F.Fab")
-			(hide yes)
-			(effects
-				(font
-					(size 1 1)
-					(thickness 0.15)
-				)
-			)
-		)
 		(property ki_fp_filters "TO-???* *_Diode_* *SingleDiode* D_*")
 		(sheetname "/")
 		(sheetfile "Main Control Unit.kicad_sch")
-		(units
-			(unit
-				(name "A")
-				(pins "1" "2")
-			)
-		)
 		(attr smd)
 		(duplicate_pad_numbers_are_jumpers no)
@@
 		(pad "1" smd roundrect
 			(at -1.1 0 90)
-			(size 0.5 0.5)
+			(size 0.75 0.75)
 			(layers "F.Cu" "F.Mask" "F.Paste")
 			(roundrect_rratio 0.25)
@@
 		(pad "2" smd roundrect
 			(at 1.1 0 90)
-			(size 0.5 0.5)
+			(size 0.75 0.75)
 			(layers "F.Cu" "F.Mask" "F.Paste")
 			(roundrect_rratio 0.25)
@@
 			)
 		)
-		(property "Datasheet" "https://assets.nexperia.com/documents/data-sheet/PZUXB_SER.pdf"
+		(property "Datasheet" ""
 			(at 0 0 90)
 			(unlocked yes)
@@
 			)
 		)
-		(property "Description" "Zener Diode 15 V 310 mW ±2% Surface Mount SOD-323F"
+		(property "Description" ""
 			(at 0 0 90)
 			(unlocked yes)
@@
 			)
 		)
-		(property "Part" "Nexperia PZU15B2,115"
-			(at 0 0 90)
-			(unlocked yes)
-			(layer "F.Fab")
-			(hide yes)
-			(effects
-				(font
-					(size 1 1)
-					(thickness 0.15)
-				)
-			)
-		)
 		(property ki_fp_filters "TO-???* *_Diode_* *SingleDiode* D_*")
 		(sheetname "/")
 		(sheetfile "Main Control Unit.kicad_sch")
-		(units
-			(unit
-				(name "A")
-				(pins "1" "2")
-			)
-		)
 		(attr smd)
 		(duplicate_pad_numbers_are_jumpers no)
@@
 		(pad "1" smd roundrect
 			(at -1.1 0 90)
-			(size 0.5 0.5)
+			(size 0.75 0.75)
 			(layers "F.Cu" "F.Mask" "F.Paste")
 			(roundrect_rratio 0.25)
@@
 		(pad "2" smd roundrect
 			(at 1.1 0 90)
-			(size 0.5 0.5)
+			(size 0.75 0.75)
 			(layers "F.Cu" "F.Mask" "F.Paste")
 			(roundrect_rratio 0.25)
@@
 			)
 		)
-		(property "Datasheet" "https://assets.nexperia.com/documents/data-sheet/PZUXB_SER.pdf"
+		(property "Datasheet" ""
 			(at 0 0 90)
 			(unlocked yes)
@@
 			)
 		)
-		(property "Description" "Zener Diode 15 V 310 mW ±2% Surface Mount SOD-323F"
+		(property "Description" ""
 			(at 0 0 90)
 			(unlocked yes)
@@
 			)
 		)
-		(property "Part" "Nexperia PZU15B2,115"
-			(at 0 0 90)
-			(unlocked yes)
-			(layer "F.Fab")
-			(hide yes)
-			(effects
-				(font
-					(size 1 1)
-					(thickness 0.15)
-				)
-			)
-		)
 		(property ki_fp_filters "TO-???* *_Diode_* *SingleDiode* D_*")
 		(sheetname "/")
 		(sheetfile "Main Control Unit.kicad_sch")
-		(units
-			(unit
-				(name "A")
-				(pins "1" "2")
-			)
-		)
 		(attr smd)
 		(duplicate_pad_numbers_are_jumpers no)
@@
 		(pad "1" smd roundrect
 			(at -1.1 0 90)
-			(size 0.5 0.5)
+			(size 0.75 0.75)
 			(layers "F.Cu" "F.Mask" "F.Paste")
 			(roundrect_rratio 0.25)
@@
 		(pad "2" smd roundrect
 			(at 1.1 0 90)
-			(size 0.5 0.5)
+			(size 0.75 0.75)
 			(layers "F.Cu" "F.Mask" "F.Paste")
 			(roundrect_rratio 0.25)
@@
 			)
 		)
-		(property "Datasheet" "https://assets.nexperia.com/documents/data-sheet/PZUXB_SER.pdf"
+		(property "Datasheet" ""
 			(at 0 0 90)
 			(unlocked yes)
@@
 			)
 		)
-		(property "Description" "Zener Diode 15 V 310 mW ±2% Surface Mount SOD-323F"
+		(property "Description" ""
 			(at 0 0 90)
 			(unlocked yes)
@@
 			)
 		)
-		(property "Part" "Nexperia PZU15B2,115"
-			(at 0 0 90)
-			(unlocked yes)
-			(layer "F.Fab")
-			(hide yes)
-			(effects
-				(font
-					(size 1 1)
-					(thickness 0.15)
-				)
-			)
-		)
 		(property ki_fp_filters "TO-???* *_Diode_* *SingleDiode* D_*")
 		(sheetname "/")
 		(sheetfile "Main Control Unit.kicad_sch")
-		(units
-			(unit
-				(name "A")
-				(pins "1" "2")
-			)
-		)
 		(attr smd)
 		(duplicate_pad_numbers_are_jumpers no)
@@
 		(pad "1" smd roundrect
 			(at -1.1 0 90)
-			(size 0.5 0.5)
+			(size 0.75 0.75)
 			(layers "F.Cu" "F.Mask" "F.Paste")
 			(roundrect_rratio 0.25)
@@
 		(pad "2" smd roundrect
 			(at 1.1 0 90)
-			(size 0.5 0.5)
+			(size 0.75 0.75)
 			(layers "F.Cu" "F.Mask" "F.Paste")
 			(roundrect_rratio 0.25)
